Commit message: [grape_with_arm] tmp urdf update for debug

File: robots/gimbalrotor/robots/grape_with_arm/gimbalrotor.gazebo.xacro (robot description, xacro)
@@ -7,3 +7,11 @@
   <xacro:include filename="$(find aerial_robot_simulation)/xacro/spinal.gazebo.xacro" />
   <xacro:gazebo_spinal robot_name="$(arg robot_name)" mag_frame="fc" />
+  <xacro:rotor_transmission id="1"/>
+  <xacro:rotor_transmission id="2"/>
+  <xacro:rotor_transmission id="3"/>
+  <xacro:rotor_transmission id="4"/>
+  <xacro:joint_transmission joint="gimbal1"/>
+  <xacro:joint_transmission joint="gimbal2"/>
+  <xacro:joint_transmission joint="gimbal3"/>
+  <xacro:joint_transmission joint="gimbal4"/>
 </robot>

File: robots/gimbalrotor/urdf/grape_with_arm/gimbalrotor.urdf.xacro (robot description, xacro)
@@ -2,6 +2,22 @@
 <robot name="gimbalrotor" xmlns:xacro="http://www.ros.org/wiki/xacro">
   <xacro:include filename="$(find gimbalrotor)/urdf/grape/common.xacro"/>
-  <xacro:include filename="$(find gimbalrotor)/urdf/grape/xacro/arm.xacro"/>
-  <link name="root">
+  <!-- <xacro:include filename="$(find gimbalrotor)/urdf/grape/xacro/arm.xacro"/> -->
+  <!-- <link name="root"> -->
+  <!--   <inertial> -->
+  <!--     <origin xyz="0 0 0" rpy="0 0 0"/> -->
+  <!--     <mass value="0.00001"/> -->
+  <!--     <inertia -->
+  <!--         ixx="0.000001" ixy="0.0" ixz="0.0" -->
+  <!--         iyy="0.000001" iyz="0.0" -->
+  <!--         izz="0.000001"/> -->
+  <!--   </inertial> -->
+  <!-- </link> -->
+  <!-- <joint name="root_joint" type="fixed"> -->
+  <!--   <parent link="root"/> -->
+  <!--   <child link="main_body"/> -->
+  <!--   <origin rpy="0 0 0" xyz="0 0 0"/> -->
+  <!--   <axis xyz="0 0 1"/> -->
+  <!-- </joint> -->
+  <link name="fc">
     <inertial>
       <origin xyz="0 0 0" rpy="0 0 0"/>
@@ -13,11 +29,11 @@
     </inertial>
   </link>
-  <joint name="root_joint" type="fixed">
-    <parent link="root"/>
-    <child link="main_body"/>
+  <joint name="fc_joint" type="fixed">
+    <child link="fc"/>
+    <parent link="main_body"/>
     <origin rpy="0 0 0" xyz="0 0 0"/>
     <axis xyz="0 0 1"/>
   </joint>
-  <link name="fc">
+  <link name="lidar_imu">
     <inertial>
       <origin xyz="0 0 0" rpy="0 0 0"/>
@@ -29,20 +45,4 @@
     </inertial>
   </link>
-  <joint name="fc_joint" type="fixed">
-    <child link="fc"/>
-    <parent link="main_body"/>
-    <origin rpy="0 0 0" xyz="0 0 0"/>
-    <axis xyz="0 0 1"/>
-  </joint>
-  <link name="lidar_imu">
-    <inertial>
-      <origin xyz="0 0 0" rpy="0 0 0"/>
-      <mass value="0.00001"/>
-      <inertia
-          ixx="0.000001" ixy="0.0" ixz="0.0"
-          iyy="0.000001" iyz="0.0"
-          izz="0.000001"/>
-    </inertial>
-  </link>
   <joint name="lidar_joint" type="fixed">
     <child link="lidar_imu"/>
@@ -184,40 +184,40 @@
     </visual>
   </link>
-  <link name="rotor_arm1">
-    <xacro:virtual_inertial/>
-  </link>
-  <link name="rotor_arm2">
-    <xacro:virtual_inertial/>
-  </link>
-  <link name="rotor_arm3">
-    <xacro:virtual_inertial/>
-  </link>
-  <link name="rotor_arm4">
-    <xacro:virtual_inertial/>
-  </link>
-  <joint name="rotor_arm1_joint" type="fixed">
-    <parent link="main_body"/>
-    <child link="rotor_arm1"/>
-    <axis xyz="0 0 1"/>
-    <origin xyz="-0.22309 -0.22309 0.0" rpy="0.0 -0.0 -2.3562"/>
-  </joint>
-  <joint name="rotor_arm2_joint" type="fixed">
-    <parent link="main_body"/>
-    <child link="rotor_arm2"/>
-    <axis xyz="0 0 1"/>
-    <origin xyz="0.22309 -0.22309 0.0" rpy="-0.0 -0.0 -0.7854000000000001"/>
-  </joint>
-  <joint name="rotor_arm3_joint" type="fixed">
-    <parent link="main_body"/>
-    <child link="rotor_arm3"/>
-    <axis xyz="0 0 1"/>
-    <origin xyz="0.22309 0.22309 0.0" rpy="0.0 -0.0 0.7854000000000001"/>
-  </joint>
-  <joint name="rotor_arm4_joint" type="fixed">
-    <parent link="main_body"/>
-    <child link="rotor_arm4"/>
-    <axis xyz="0 0 1"/>
-    <origin xyz="-0.22309 0.22309 0.0" rpy="0.0 -0.0 2.3562"/>
-  </joint>
+  <!-- <link name="rotor_arm1"> -->
+  <!--   <xacro:virtual_inertial/> -->
+  <!-- </link> -->
+  <!-- <link name="rotor_arm2"> -->
+  <!--   <xacro:virtual_inertial/> -->
+  <!-- </link> -->
+  <!-- <link name="rotor_arm3"> -->
+  <!--   <xacro:virtual_inertial/> -->
+  <!-- </link> -->
+  <!-- <link name="rotor_arm4"> -->
+  <!--   <xacro:virtual_inertial/> -->
+  <!-- </link> -->
+  <!-- <joint name="rotor_arm1_joint" type="fixed"> -->
+  <!--   <parent link="main_body"/> -->
+  <!--   <child link="rotor_arm1"/> -->
+  <!--   <axis xyz="0 0 1"/> -->
+  <!--   <origin xyz="-0.22309 -0.22309 0.0" rpy="0.0 -0.0 -2.3562"/> -->
+  <!-- </joint> -->
+  <!-- <joint name="rotor_arm2_joint" type="fixed"> -->
+  <!--   <parent link="main_body"/> -->
+  <!--   <child link="rotor_arm2"/> -->
+  <!--   <axis xyz="0 0 1"/> -->
+  <!--   <origin xyz="0.22309 -0.22309 0.0" rpy="-0.0 -0.0 -0.7854000000000001"/> -->
+  <!-- </joint> -->
+  <!-- <joint name="rotor_arm3_joint" type="fixed"> -->
+  <!--   <parent link="main_body"/> -->
+  <!--   <child link="rotor_arm3"/> -->
+  <!--   <axis xyz="0 0 1"/> -->
+  <!--   <origin xyz="0.22309 0.22309 0.0" rpy="0.0 -0.0 0.7854000000000001"/> -->
+  <!-- </joint> -->
+  <!-- <joint name="rotor_arm4_joint" type="fixed"> -->
+  <!--   <parent link="main_body"/> -->
+  <!--   <child link="rotor_arm4"/> -->
+  <!--   <axis xyz="0 0 1"/> -->
+  <!--   <origin xyz="-0.22309 0.22309 0.0" rpy="0.0 -0.0 2.3562"/> -->
+  <!-- </joint> -->
   <joint name="gimbal1" type="revolute">
     <limit effort="5.0" velocity="10.0" lower="-3.14" upper="3.14"/>
@@ -316,44 +316,44 @@
     </actuator>
   </transmission>
-    <transmission name="rotor_tran1">
-      <type>transmission_interface/SimpleTransmission</type>
-      <joint name="rotor1">
-        <hardwareInterface>RotorInterface</hardwareInterface>
-      </joint>
-      <actuator name="rotor_actuator1">
-        <hardwareInterface>RotorInterface</hardwareInterface>
-        <mechanicalReduction>1</mechanicalReduction>
-      </actuator>
-    </transmission>
-    <transmission name="rotor_tran2">
-      <type>transmission_interface/SimpleTransmission</type>
-      <joint name="rotor2">
-        <hardwareInterface>RotorInterface</hardwareInterface>
-      </joint>
-      <actuator name="rotor_actuator2">
-        <hardwareInterface>RotorInterface</hardwareInterface>
-        <mechanicalReduction>1</mechanicalReduction>
-      </actuator>
-    </transmission>
-    <transmission name="rotor_tran3">
-      <type>transmission_interface/SimpleTransmission</type>
-      <joint name="rotor3">
-        <hardwareInterface>RotorInterface</hardwareInterface>
-      </joint>
-      <actuator name="rotor_actuator3">
-        <hardwareInterface>RotorInterface</hardwareInterface>
-        <mechanicalReduction>1</mechanicalReduction>
-      </actuator>
-    </transmission>
-    <transmission name="rotor_tran4">
-      <type>transmission_interface/SimpleTransmission</type>
-      <joint name="rotor4">
-        <hardwareInterface>RotorInterface</hardwareInterface>
-      </joint>
-      <actuator name="rotor_actuator4">
-        <hardwareInterface>RotorInterface</hardwareInterface>
-        <mechanicalReduction>1</mechanicalReduction>
-      </actuator>
-    </transmission>
+  <transmission name="rotor_tran1">
+    <type>transmission_interface/SimpleTransmission</type>
+    <joint name="rotor1">
+      <hardwareInterface>RotorInterface</hardwareInterface>
+    </joint>
+    <actuator name="rotor_actuator1">
+      <hardwareInterface>RotorInterface</hardwareInterface>
+      <mechanicalReduction>1</mechanicalReduction>
+    </actuator>
+  </transmission>
+  <transmission name="rotor_tran2">
+    <type>transmission_interface/SimpleTransmission</type>
+    <joint name="rotor2">
+      <hardwareInterface>RotorInterface</hardwareInterface>
+    </joint>
+    <actuator name="rotor_actuator2">
+      <hardwareInterface>RotorInterface</hardwareInterface>
+      <mechanicalReduction>1</mechanicalReduction>
+    </actuator>
+  </transmission>
+  <transmission name="rotor_tran3">
+    <type>transmission_interface/SimpleTransmission</type>
+    <joint name="rotor3">
+      <hardwareInterface>RotorInterface</hardwareInterface>
+    </joint>
+    <actuator name="rotor_actuator3">
+      <hardwareInterface>RotorInterface</hardwareInterface>
+      <mechanicalReduction>1</mechanicalReduction>
+    </actuator>
+  </transmission>
+  <transmission name="rotor_tran4">
+    <type>transmission_interface/SimpleTransmission</type>
+    <joint name="rotor4">
+      <hardwareInterface>RotorInterface</hardwareInterface>
+    </joint>
+    <actuator name="rotor_actuator4">
+      <hardwareInterface>RotorInterface</hardwareInterface>
+      <mechanicalReduction>1</mechanicalReduction>
+    </actuator>
+  </transmission>
   <material name="__unnamed_material_1">
     <color rgba="0.10980392 0.10980392 0.10980392 1.        "/>
@@ -383,5 +383,20 @@
     <color rgba="0.50196078 0.50196078 0.50196078 1.        "/>
   </material>
+  <link name="battery">
+    <inertial>
+      <origin xyz="0 0 0" rpy="0 0 0"/>
+      <mass value="1.1"/>
+      <inertia
+          ixx="0.0012" ixy="0.0" ixz="0.0"
+          iyy="0.0012" iyz="0.0"
+          izz="0.0012"/>
+    </inertial>
+  </link>
+  <joint name="battery_joint" type="fixed">
+    <parent link="main_body"/>
+    <child link="battery"/>
+    <origin xyz="0 0 -0.08" rpy="3.14159 0 0"/>
+  </joint>
   <!-- Include the arm macro -->
-  <xacro:arm parent_link="main_body"/>
+  <!-- <xacro:arm parent_link="main_body"/> -->
 </robot>
