Commit message: [grape_with_arm] add arm

File: robots/gimbalrotor/urdf/grape/xacro/screw_200mmpipe_module.xacro (robot description, xacro)
@@ -20,10 +20,10 @@
         <origin xyz="-0.018612068965513 1.00000000000001 0.146669004611067" rpy="-1.5707963267948835 1.570796326794893 3.141592653589793"/>
       </visual>
-      <collision>
-        <geometry>
-          <mesh filename="package://${package_name}/urdf/grape/meshes/arm/screw_200mmpipe_module/base_link.stl"/>
-        </geometry>
-        <origin xyz="-0.018612068965513 1.00000000000001 0.146669004611067" rpy="-1.5707963267948835 1.570796326794893 3.141592653589793"/>
-      </collision>
+      <!-- <collision> -->
+      <!--   <geometry> -->
+      <!--     <mesh filename="package://${package_name}/urdf/grape/meshes/arm/screw_200mmpipe_module/base_link.stl"/> -->
+      <!--   </geometry> -->
+      <!--   <origin xyz="-0.018612068965513 1.00000000000001 0.146669004611067" rpy="-1.5707963267948835 1.570796326794893 3.141592653589793"/> -->
+      <!-- </collision> -->
     </link>
     <link name="${prefix}dummy_link"/>

File: robots/gimbalrotor/urdf/grape/xacro/screw_90deg_module.xacro (robot description, xacro)
@@ -20,10 +20,10 @@
         <origin xyz="0.0285 -1.88586037787625e-16 0.0285000000000001" rpy="3.14159265358979 -2.52653528463934e-16 1.57079632679489"/>
       </visual>
-      <collision>
-        <geometry>
-          <mesh filename="package://${package_name}/urdf/grape/meshes/arm/screw_90deg_module/base_link.dae"/>
-        </geometry>
-        <origin xyz="0.0285 -1.88586037787625e-16 0.0285000000000001" rpy="3.14159265358979 -2.52653528463934e-16 1.57079632679489"/>
-      </collision>
+      <!-- <collision> -->
+      <!--   <geometry> -->
+      <!--     <mesh filename="package://${package_name}/urdf/grape/meshes/arm/screw_90deg_module/base_link.dae"/> -->
+      <!--   </geometry> -->
+      <!--   <origin xyz="0.0285 -1.88586037787625e-16 0.0285000000000001" rpy="3.14159265358979 -2.52653528463934e-16 1.57079632679489"/> -->
+      <!-- </collision> -->
     </link>
     <link name="${prefix}dummy_link"/>

File: robots/gimbalrotor/urdf/grape/xacro/screw_drive_module_dynamixel.xacro (robot description, xacro)
@@ -20,10 +20,10 @@
         <origin xyz="-1.51387102717471e-18 5.99174275367398e-19 0.0457" rpy="1.5707963267949003 -0.0 1.5707963267949003"/>
       </visual>
-      <collision>
-        <geometry>
-          <mesh filename="package://${package_name}/urdf/grape/meshes/arm/screw_drive_module_dynamixel/base_link.stl"/>
-        </geometry>
-        <origin xyz="-1.51387102717471e-18 5.99174275367398e-19 0.0457" rpy="1.5707963267949003 -0.0 1.5707963267949003"/>
-      </collision>
+      <!-- <collision> -->
+      <!--   <geometry> -->
+      <!--     <mesh filename="package://${package_name}/urdf/grape/meshes/arm/screw_drive_module_dynamixel/base_link.stl"/> -->
+      <!--   </geometry> -->
+      <!--   <origin xyz="-1.51387102717471e-18 5.99174275367398e-19 0.0457" rpy="1.5707963267949003 -0.0 1.5707963267949003"/> -->
+      <!-- </collision> -->
     </link>
     <link name="${prefix}link1">
@@ -40,10 +40,10 @@
         <origin xyz="-2.15167357330528e-17 -1.20100411619191e-17 0.0152" rpy="1.5707963267949003 -1.09476442525376e-47 1.5707963267949003"/>
       </visual>
-      <collision>
-        <geometry>
-          <mesh filename="package://${package_name}/urdf/grape/meshes/arm/screw_drive_module_dynamixel/link1.stl"/>
-        </geometry>
-        <origin xyz="-2.15167357330528e-17 -1.20100411619191e-17 0.0152" rpy="1.5707963267949003 -1.09476442525376e-47 1.5707963267949003"/>
-      </collision>
+      <!-- <collision> -->
+      <!--   <geometry> -->
+      <!--     <mesh filename="package://${package_name}/urdf/grape/meshes/arm/screw_drive_module_dynamixel/link1.stl"/> -->
+      <!--   </geometry> -->
+      <!--   <origin xyz="-2.15167357330528e-17 -1.20100411619191e-17 0.0152" rpy="1.5707963267949003 -1.09476442525376e-47 1.5707963267949003"/> -->
+      <!-- </collision> -->
     </link>
     <link name="${prefix}dummy_link"/>

File: robots/gimbalrotor/urdf/grape/xacro/screw_hinge_module_dynamixel.xacro (robot description, xacro)
@@ -20,10 +20,10 @@
         <origin xyz="0.0 0.0 0.0" rpy="1.5707963267949003 -2.99239799605999e-16 -1.5707963267949003"/>
       </visual>
-      <collision>
-        <geometry>
-          <mesh filename="package://${package_name}/urdf/grape/meshes/arm/screw_hinge_module_dynamixel/base_link.stl"/>
-        </geometry>
-        <origin xyz="0.0 0.0 0.0" rpy="1.5707963267949003 -2.99239799605999e-16 -1.5707963267949003"/>
-      </collision>
+      <!-- <collision> -->
+      <!--   <geometry> -->
+      <!--     <mesh filename="package://${package_name}/urdf/grape/meshes/arm/screw_hinge_module_dynamixel/base_link.stl"/> -->
+      <!--   </geometry> -->
+      <!--   <origin xyz="0.0 0.0 0.0" rpy="1.5707963267949003 -2.99239799605999e-16 -1.5707963267949003"/> -->
+      <!-- </collision> -->
     </link>
     <link name="${prefix}link1">
@@ -40,10 +40,10 @@
         <origin xyz="2.09657352239695e-18 -0.035 1.00064680020069e-17" rpy="3.141592653589793 1.570796326794893 3.141592653589793"/>
       </visual>
-      <collision>
-        <geometry>
-          <mesh filename="package://${package_name}/urdf/grape/meshes/arm/screw_hinge_module_dynamixel/link1.stl"/>
-        </geometry>
-        <origin xyz="2.09657352239695e-18 -0.035 1.00064680020069e-17" rpy="3.141592653589793 1.570796326794893 3.141592653589793"/>
-      </collision>
+      <!-- <collision> -->
+      <!--   <geometry> -->
+      <!--     <mesh filename="package://${package_name}/urdf/grape/meshes/arm/screw_hinge_module_dynamixel/link1.stl"/> -->
+      <!--   </geometry> -->
+      <!--   <origin xyz="2.09657352239695e-18 -0.035 1.00064680020069e-17" rpy="3.141592653589793 1.570796326794893 3.141592653589793"/> -->
+      <!-- </collision> -->
     </link>
     <link name="${prefix}dummy_link"/>

File: robots/gimbalrotor/urdf/grape/xacro/screw_yaw_module_dynamixel_side.xacro (robot description, xacro)
@@ -20,10 +20,10 @@
         <origin xyz="0.0 0.0 0.0" rpy="1.5707963267949003 2.83742224257185e-17 5.37764277552873e-17"/>
       </visual>
-      <collision>
-        <geometry>
-          <mesh filename="package://${package_name}/urdf/grape/meshes/arm/screw_yaw_module_dynamixel_side/base_link.stl"/>
-        </geometry>
-        <origin xyz="0.0 0.0 0.0" rpy="1.5707963267949003 2.83742224257185e-17 5.37764277552873e-17"/>
-      </collision>
+      <!-- <collision> -->
+      <!--   <geometry> -->
+      <!--     <mesh filename="package://${package_name}/urdf/grape/meshes/arm/screw_yaw_module_dynamixel_side/base_link.stl"/> -->
+      <!--   </geometry> -->
+      <!--   <origin xyz="0.0 0.0 0.0" rpy="1.5707963267949003 2.83742224257185e-17 5.37764277552873e-17"/> -->
+      <!-- </collision> -->
     </link>
     <link name="${prefix}link1">
@@ -40,10 +40,10 @@
         <origin xyz="-0.00399999999999988 1.52187655629222e-16 -0.0285" rpy="1.5707963267949003 6.48786257890944e-17 -1.5707963267949003"/>
       </visual>
-      <collision>
-        <geometry>
-          <mesh filename="package://${package_name}/urdf/grape/meshes/arm/screw_yaw_module_dynamixel_side/link1.stl"/>
-        </geometry>
-        <origin xyz="-0.00399999999999988 1.52187655629222e-16 -0.0285" rpy="1.5707963267949003 6.48786257890944e-17 -1.5707963267949003"/>
-      </collision>
+      <!-- <collision> -->
+      <!--   <geometry> -->
+      <!--     <mesh filename="package://${package_name}/urdf/grape/meshes/arm/screw_yaw_module_dynamixel_side/link1.stl"/> -->
+      <!--   </geometry> -->
+      <!--   <origin xyz="-0.00399999999999988 1.52187655629222e-16 -0.0285" rpy="1.5707963267949003 6.48786257890944e-17 -1.5707963267949003"/> -->
+      <!-- </collision> -->
     </link>
     <link name="${prefix}dummy_link"/>

File: robots/gimbalrotor/urdf/grape/xacro/vial_pick_module.xacro (robot description, xacro)
@@ -20,10 +20,10 @@
         <origin xyz="0.0 0.0 0.0" rpy="-1.1895621213035508e-32 -2.44929359829471e-16 1.57079632679489"/>
       </visual>
-      <collision>
-        <geometry>
-          <mesh filename="package://${package_name}/urdf/grape/meshes/arm/vial_pick_module/base_link.stl"/>
-        </geometry>
-        <origin xyz="0.0 0.0 0.0" rpy="-1.1895621213035508e-32 -2.44929359829471e-16 1.57079632679489"/>
-      </collision>
+      <!-- <collision> -->
+      <!--   <geometry> -->
+      <!--     <mesh filename="package://${package_name}/urdf/grape/meshes/arm/vial_pick_module/base_link.stl"/> -->
+      <!--   </geometry> -->
+      <!--   <origin xyz="0.0 0.0 0.0" rpy="-1.1895621213035508e-32 -2.44929359829471e-16 1.57079632679489"/> -->
+      <!-- </collision> -->
     </link>
     <link name="${prefix}pick_dummy_link">
@@ -40,10 +40,10 @@
         <origin xyz="-1.43008831174061e-17 -1.78863404261684e-17 -0.023" rpy="-1.3497194182685498e-15 -7.618871916663648e-16 -1.5707963267944498"/>
       </visual>
-      <collision>
-        <geometry>
-          <mesh filename="package://${package_name}/urdf/grape/meshes/arm/vial_pick_module/pick_dummy_link.stl"/>
-        </geometry>
-        <origin xyz="-1.43008831174061e-17 -1.78863404261684e-17 -0.023" rpy="-1.3497194182685498e-15 -7.618871916663648e-16 -1.5707963267944498"/>
-      </collision>
+      <!-- <collision> -->
+      <!--   <geometry> -->
+      <!--     <mesh filename="package://${package_name}/urdf/grape/meshes/arm/vial_pick_module/pick_dummy_link.stl"/> -->
+      <!--   </geometry> -->
+      <!--   <origin xyz="-1.43008831174061e-17 -1.78863404261684e-17 -0.023" rpy="-1.3497194182685498e-15 -7.618871916663648e-16 -1.5707963267944498"/> -->
+      <!-- </collision> -->
     </link>
     <link name="${prefix}gripper_link1">
@@ -60,10 +60,10 @@
         <origin xyz="-0.00699999999999998 1.0683109299301e-18 -0.0235" rpy="6.301392866405062e-16 -9.87992243989157e-16 -1.5707963267949006"/>
       </visual>
-      <collision>
-        <geometry>
-          <mesh filename="package://${package_name}/urdf/grape/meshes/arm/vial_pick_module/gripper_link1.stl"/>
-        </geometry>
-        <origin xyz="-0.00699999999999998 1.0683109299301e-18 -0.0235" rpy="6.301392866405062e-16 -9.87992243989157e-16 -1.5707963267949006"/>
-      </collision>
+      <!-- <collision> -->
+      <!--   <geometry> -->
+      <!--     <mesh filename="package://${package_name}/urdf/grape/meshes/arm/vial_pick_module/gripper_link1.stl"/> -->
+      <!--   </geometry> -->
+      <!--   <origin xyz="-0.00699999999999998 1.0683109299301e-18 -0.0235" rpy="6.301392866405062e-16 -9.87992243989157e-16 -1.5707963267949006"/> -->
+      <!-- </collision> -->
     </link>
     <link name="${prefix}gripper_link2">
@@ -80,10 +80,10 @@
         <origin xyz="0.00700000000000003 1.31857538436738e-16 -0.0235" rpy="5.703715567474983e-16 -1.04683580036436e-15 -1.5707963267949006"/>
       </visual>
-      <collision>
-        <geometry>
-          <mesh filename="package://${package_name}/urdf/grape/meshes/arm/vial_pick_module/gripper_link2.stl"/>
-        </geometry>
-        <origin xyz="0.00700000000000003 1.31857538436738e-16 -0.0235" rpy="5.703715567474983e-16 -1.04683580036436e-15 -1.5707963267949006"/>
-      </collision>
+      <!-- <collision> -->
+      <!--   <geometry> -->
+      <!--     <mesh filename="package://${package_name}/urdf/grape/meshes/arm/vial_pick_module/gripper_link2.stl"/> -->
+      <!--   </geometry> -->
+      <!--   <origin xyz="0.00700000000000003 1.31857538436738e-16 -0.0235" rpy="5.703715567474983e-16 -1.04683580036436e-15 -1.5707963267949006"/> -->
+      <!-- </collision> -->
     </link>
     <joint name="${prefix}pick_dummy_joint" type="revolute">

File: robots/gimbalrotor/urdf/grape_with_arm/gimbalrotor.urdf.xacro (robot description, xacro)
@@ -2,5 +2,5 @@
 <robot name="gimbalrotor" xmlns:xacro="http://www.ros.org/wiki/xacro">
   <xacro:include filename="$(find gimbalrotor)/urdf/grape/common.xacro"/>
-  <!-- <xacro:include filename="$(find gimbalrotor)/urdf/grape/xacro/arm.xacro"/> -->
+  <xacro:include filename="$(find gimbalrotor)/urdf/grape/xacro/arm.xacro"/>
   <!-- <link name="root"> -->
   <!--   <inertial> -->
@@ -399,4 +399,4 @@
   </joint>
   <!-- Include the arm macro -->
-  <!-- <xacro:arm parent_link="main_body"/> -->
+  <xacro:arm parent_link="main_body"/>
 </robot>
