Commit message: [gimbalrotor] update URDF and bringup.launch

File: robots/gimbalrotor/urdf/grape/xacro/arm.xacro (robot description, xacro)
@@ -51,7 +51,12 @@
       xyz="0 0 0"
       rpy="0 3.14 0"/>
+    <!-- <xacro:screw_hinge_module_dynamixel -->
+    <!--   prefix="arm_joint5_" -->
+    <!--   parent_link="arm_joint4_dummy_link" -->
+    <!--   xyz="0 0 0" -->
+    <!--   rpy="0 3.14 0"/> -->
     <!-- Joint 5: Drive module -->
     <xacro:screw_drive_module_dynamixel
-      prefix="arm_joint5_"
+	prefix="arm_joint5_"
       parent_link="arm_joint4_dummy_link"
       xyz="0 0 0"
@@ -61,4 +66,5 @@
       prefix="arm_gripper_"
       parent_link="arm_joint5_dummy_link"
+      parent_joint="arm_joint5_joint1"
       xyz="0 0 0"
       rpy="0 0 0"/>

File: robots/gimbalrotor/urdf/grape/xacro/screw_drive_module_dynamixel.xacro (robot description, xacro)
@@ -32,4 +32,8 @@
         <mass value="0.00140627867032843"/>
         <inertia ixx="3.69305972647323e-08" ixy="4.70059675645385e-16" ixz="1.36569540430659e-09" iyy="4.37001527382599e-08" iyz="4.21205301040001e-16" izz="6.37416918942377e-08"/>
+	<!-- <mass value="0.00000001"/> -->
+	<!-- <inertia ixx="1e-10" ixy="1e-10" ixz="1e-10" -->
+	<!-- 	 iyy="1e-10" iyz="1e-10" -->
+	<!-- 	 izz="1e-10"/> -->
       </inertial>
       <visual>
@@ -48,10 +52,15 @@
     </link>
     <link name="${prefix}dummy_link"/>
-    <joint name="${prefix}joint1" type="continuous">
-      <limit effort="0.0" velocity="0.0"/>
+    <joint name="${prefix}joint1" type="revolute">
+      <!-- <joint name="${prefix}joint1" type="continuous"> -->
+      <!-- <limit effort="1.5" velocity="6.39"/> -->
+      <!-- <limit effort="300" velocity="6.39" lower="-3.141592" upper="3.141592"/> -->
+      <limit effort="1.5" velocity="6.39" lower="-3.141592" upper="3.141592"/>
+      <!-- <limit effort="0.0" velocity="0.0"/> -->
       <parent link="${prefix}base_link"/>
       <child link="${prefix}link1"/>
       <axis xyz=" 0.  0. -1."/>
       <origin xyz="0.0 0.0 0.0305" rpy="0.0 -0.0 0.0"/>
+      <dynamics damping="0.000001" friction="0.0000001"/>
     </joint>
     <joint name="${prefix}dummy_joint" type="fixed">

File: robots/gimbalrotor/urdf/grape/xacro/screw_hinge_module_dynamixel.xacro (robot description, xacro)
@@ -49,5 +49,6 @@
     <link name="${prefix}dummy_link"/>
     <joint name="${prefix}joint1" type="revolute">
-      <limit effort="0.0" velocity="0.0" lower="-3.141592" upper="3.141592"/>
+      <limit effort="1.5" velocity="6.39" lower="-3.141592" upper="3.141592"/>
+      <!-- <limit effort="0.0" velocity="0.0" lower="-3.141592" upper="3.141592"/> -->
       <!-- <limit effort="0.0" velocity="0.0" lower="-0.567" upper="0.567"/> -->
       <parent link="${prefix}base_link"/>

File: robots/gimbalrotor/urdf/grape/xacro/screw_yaw_module_dynamixel_side.xacro (robot description, xacro)
@@ -49,5 +49,6 @@
     <link name="${prefix}dummy_link"/>
     <joint name="${prefix}joint1" type="revolute">
-      <limit effort="0.0" velocity="0.0" lower="-3.14" upper="3.14"/>
+      <limit effort="3.0" velocity="8.06" lower="-3.14" upper="3.14"/>
+      <!-- <limit effort="0.0" velocity="0.0" lower="-3.14" upper="3.14"/> -->
       <parent link="${prefix}base_link"/>
       <child link="${prefix}link1"/>

File: robots/gimbalrotor/urdf/grape/xacro/vial_pick_module.xacro (robot description, xacro)
@@ -1,5 +1,5 @@
 <?xml version='1.0' encoding='UTF-8'?>
 <robot xmlns:xacro="http://ros.org/wiki/xacro" name="vial_pick_module">
-  <xacro:macro name="vial_pick_module" params="prefix:='' parent_link:=world xyz:='0 0 0' rpy:='0 0 0' package_name:=gimbalrotor">
+  <xacro:macro name="vial_pick_module" params="prefix:='' parent_link:=world xyz:='0 0 0' rpy:='0 0 0' package_name:=gimbalrotor parent_joint:=''">
     <joint name="${parent_link}_to_${prefix}base_link_joint" type="fixed">
       <parent link="${parent_link}"/>
@@ -88,5 +88,7 @@
     </link>
     <joint name="${prefix}pick_dummy_joint" type="revolute">
-      <limit effort="0.0" velocity="0.0" lower="-2.36" upper="2.36"/>
+      <limit effort="1.5" velocity="6.0" lower="-2.36" upper="2.36"/>
+      <mimic joint="${parent_joint}" multiplier="-1" offset="0.0"/>
+      <!-- <mimic joint="arm_joint5_joint1" multiplier="1" offset="0.0"/> -->
       <parent link="${prefix}base_link"/>
       <child link="${prefix}pick_dummy_link"/>
@@ -95,6 +97,7 @@
     </joint>
     <joint name="${prefix}gripper_joint1" type="prismatic">
-      <limit effort="0.0" velocity="0.0" lower="-0.013" upper="0.018"/>
-      <mimic joint="${prefix}pick_dummy_joint" multiplier="-0.007" offset="0.0"/>
+      <limit effort="1.5" velocity="6.0" lower="-0.013" upper="0.018"/>
+      <!-- <mimic joint="${prefix}pick_dummy_joint" multiplier="-0.007" offset="0.0"/> -->
+      <mimic joint="${parent_joint}" multiplier="-0.007" offset="0.0"/>
       <parent link="${prefix}base_link"/>
       <child link="${prefix}gripper_link1"/>
@@ -103,6 +106,7 @@
     </joint>
     <joint name="${prefix}gripper_joint2" type="prismatic">
-      <limit effort="0.0" velocity="0.0" lower="-0.013" upper="0.018"/>
-      <mimic joint="${prefix}pick_dummy_joint" multiplier="-0.007" offset="0.0"/>
+      <limit effort="1.5" velocity="6.0" lower="-0.013" upper="0.018"/>
+      <!-- <mimic joint="${prefix}pick_dummy_joint" multiplier="-0.007" offset="0.0"/> -->
+      <mimic joint="${parent_joint}" multiplier="-0.007" offset="0.0"/>
       <parent link="${prefix}base_link"/>
       <child link="${prefix}gripper_link2"/>
