Commit message: [grape_with_arm] update mass paramators

File: robots/gimbalrotor/urdf/grape_with_arm/gimbalrotor.urdf.xacro (robot description, xacro)
@@ -54,6 +54,14 @@
     <inertial>
       <origin xyz="-0.0041019 0.0000721 -0.0183334" rpy="0.0 -0.0 0.0"/>
-      <mass value="1.3193189"/>
-      <inertia ixx="0.0150906" ixy="-0.0000095" ixz="-0.0001112" iyy="0.0153469" iyz="-0.0000102" izz="0.0122100"/>
+      <!-- <mass value="1.3193189"/> -->
+      <mass value="2.0421872"/>
+      <!-- <inertia ixx="0.0150906" ixy="-0.0000095" ixz="-0.0001112" iyy="0.0153469" iyz="-0.0000102" izz="0.0122100"/> -->
+      <inertia
+	  ixx="0.0233589"
+	  ixy="-0.0000147"
+	  ixz="-0.0001721"
+	  iyy="0.0237556"
+	  iyz="-0.0000158"
+	  izz="0.0189000"/>
     </inertial>
     <visual>
@@ -89,5 +97,6 @@
     <inertial>
       <origin xyz="-5.83353443328605e-09 6.00431360659234e-10 0.00419839092547531" rpy="0.0 -0.0 0.0"/>
-      <mass value="0.011379798689915"/>
+      <!-- <mass value="0.011379798689915"/> -->
+      <mass value="0.0247"/>
       <inertia ixx="8.74001997923959e-05" ixy="-4.12766506878745e-06" ixz="-1.94275247125274e-13" iyy="6.72594264513234e-07" iyz="8.34517033335333e-15" izz="8.79093348597008e-05"/>
     </inertial>
@@ -117,5 +126,6 @@
     <inertial>
       <origin xyz="-2.56972954026935e-09 3.06808817088874e-09 0.00419843813014376" rpy="0.0 -0.0 0.0"/>
-      <mass value="0.0113800668107397"/>
+      <!-- <mass value="0.0113800668107397"/> -->
+      <mass value="0.0247"/>
       <inertia ixx="8.73993574758916e-05" ixy="4.12756893234927e-06" ixz="-1.16071744831874e-13" iyy="6.7258088785491e-07" iyz="1.27017867936525e-13" izz="8.79084828385424e-05"/>
     </inertial>
@@ -145,5 +155,6 @@
     <inertial>
       <origin xyz="-5.83425141531535e-09 6.01800406659052e-10 0.00419839092622981" rpy="0.0 -0.0 0.0"/>
-      <mass value="0.0113797986875362"/>
+      <!-- <mass value="0.0113797986875362"/> -->
+      <mass value="0.0247"/>
       <inertia ixx="8.74001997906142e-05" ixy="-4.12766506892759e-06" ixz="-1.9423641282498e-13" iyy="6.72594264594888e-07" iyz="8.63468898765394e-15" izz="8.79093348579925e-05"/>
     </inertial>
@@ -173,5 +184,6 @@
     <inertial>
       <origin xyz="-2.5501448175369e-09 3.18832430420899e-09 0.00419843814009516" rpy="0.0 -0.0 0.0"/>
-      <mass value="0.0113800667770834"/>
+      <!-- <mass value="0.0113800667770834"/> -->
+      <mass value="0.0247"/>
       <inertia ixx="8.73993574510469e-05" ixy="4.12756894375054e-06" ixz="-1.15301708553968e-13" iyy="6.7258088604331e-07" iyz="1.31787422616219e-13" izz="8.79084828126607e-05"/>
     </inertial>
@@ -383,19 +395,19 @@
     <color rgba="0.50196078 0.50196078 0.50196078 1.        "/>
   </material>
-  <link name="battery">
-    <inertial>
-      <origin xyz="0 0 0" rpy="0 0 0"/>
-      <mass value="1.1"/>
-      <inertia
-          ixx="0.0012" ixy="0.0" ixz="0.0"
-          iyy="0.0012" iyz="0.0"
-          izz="0.0012"/>
-    </inertial>
-  </link>
-  <joint name="battery_joint" type="fixed">
-    <parent link="main_body"/>
-    <child link="battery"/>
-    <origin xyz="0 0 -0.08" rpy="3.14159 0 0"/>
-  </joint>
+  <!-- <link name="battery"> -->
+  <!--   <inertial> -->
+  <!--     <origin xyz="0 0 0" rpy="0 0 0"/> -->
+  <!--     <mass value="1.1"/> -->
+  <!--     <inertia -->
+  <!--         ixx="0.0012" ixy="0.0" ixz="0.0" -->
+  <!--         iyy="0.0012" iyz="0.0" -->
+  <!--         izz="0.0012"/> -->
+  <!--   </inertial> -->
+  <!-- </link> -->
+  <!-- <joint name="battery_joint" type="fixed"> -->
+  <!--   <parent link="main_body"/> -->
+  <!--   <child link="battery"/> -->
+  <!--   <origin xyz="0 0 -0.08" rpy="3.14159 0 0"/> -->
+  <!-- </joint> -->
   <!-- Include the arm macro -->
   <xacro:arm parent_link="main_body"/>

File: robots/gimbalrotor/urdf/grape_with_arm/xacro/screw_200mmpipe_module.xacro (robot description, xacro)
@@ -10,5 +10,6 @@
       <inertial>
         <origin xyz="0.0314472120441254 0.0185600648406693 0.999996863971173" rpy="0.0 -0.0 0.0"/>
-        <mass value="0.0784"/>
+        <!-- <mass value="0.0784"/> -->
+	<mass value="0.0807"/>
         <inertia ixx="1.92067336342704e-05" ixy="4.86844738251007e-08" ixz="-3.58103918098541e-08" iyy="0.000556258110321859" iyz="-3.52324723813976e-10" izz="0.000556910936857427"/>
       </inertial>

File: robots/gimbalrotor/urdf/grape_with_arm/xacro/screw_90deg_module.xacro (robot description, xacro)
@@ -10,5 +10,6 @@
       <inertial>
         <origin xyz="0.0103968242657149 9.09918637167594e-06 0.0216864027648383" rpy="0.0 -0.0 0.0"/>
-        <mass value="0.0326146601839408"/>
+        <!-- <mass value="0.0326146601839408"/> -->
+	<mass value="0.0387"/>
         <inertia ixx="7.31440757794881e-06" ixy="1.87744826133299e-09" ixz="-3.64840488298395e-07" iyy="5.22875275247874e-06" iyz="1.92378635215547e-09" izz="6.19875400864727e-06"/>
       </inertial>

File: robots/gimbalrotor/urdf/grape_with_arm/xacro/screw_drive_module_dynamixel.xacro (robot description, xacro)
@@ -10,5 +10,6 @@
       <inertial>
         <origin xyz="-0.00765228787056842 -4.62071402854722e-06 0.030577013511963" rpy="0.0 -0.0 0.0"/>
-        <mass value="0.0789612388386658"/>
+        <!-- <mass value="0.0789612388386658"/> -->
+	<mass value="0.10090"/>
         <inertia ixx="1.79587389811886e-05" ixy="-4.55577944240825e-09" ixz="-4.90809821784595e-07" iyy="2.50354890172928e-05" iyz="-4.43481793491922e-09" izz="2.37470837281577e-05"/>
       </inertial>
@@ -30,5 +31,6 @@
       <inertial>
         <origin xyz="-0.000256062171402636 -1.23464794906739e-10 0.0223133729686151" rpy="0.0 -0.0 0.0"/>
-        <mass value="0.00140627867032843"/>
+        <!-- <mass value="0.00140627867032843"/> -->
+	<mass value="0.0017970"/>
         <inertia ixx="3.69305972647323e-08" ixy="4.70059675645385e-16" ixz="1.36569540430659e-09" iyy="4.37001527382599e-08" iyz="4.21205301040001e-16" izz="6.37416918942377e-08"/>
 	<!-- <mass value="0.00000001"/> -->

File: robots/gimbalrotor/urdf/grape_with_arm/xacro/screw_hinge_module_dynamixel.xacro (robot description, xacro)
@@ -10,5 +10,6 @@
       <inertial>
         <origin xyz="-0.000125522807867996 6.25397854935558e-05 0.0152522387170004" rpy="0.0 -0.0 0.0"/>
-        <mass value="0.0138575446641172"/>
+        <!-- <mass value="0.0138575446641172"/> -->
+	<mass value="0.0173472031975398"/>
         <inertia ixx="3.55557358743012e-06" ixy="6.50933428796727e-10" ixz="4.46136622179202e-08" iyy="6.32031958633877e-06" iyz="-1.9253050825893e-08" izz="4.57885870672051e-06"/>
       </inertial>
@@ -30,5 +31,6 @@
       <inertial>
         <origin xyz="0.000338644241900288 0.0191313185456315 5.78940488087729e-07" rpy="0.0 -0.0 0.0"/>
-        <mass value="0.0612328998065947"/>
+        <!-- <mass value="0.0612328998065947"/> -->
+	<mass value="0.0766527968024602"/>
         <inertia ixx="1.33040989290318e-05" ixy="2.5040849060523e-07" ixz="4.80025662292933e-09" iyy="1.27387024978889e-05" iyz="-4.2924245435293e-09" izz="1.50538962870715e-05"/>
       </inertial>

File: robots/gimbalrotor/urdf/grape_with_arm/xacro/screw_yaw_module_dynamixel_side.xacro (robot description, xacro)
@@ -10,5 +10,6 @@
       <inertial>
         <origin xyz="2.05400538280698e-06 0.00964614213009143 0.0328157127384981" rpy="0.0 -0.0 0.0"/>
-        <mass value="0.0974969477576165"/>
+        <!-- <mass value="0.0974969477576165"/> -->
+	<mass value="0.134835603611421"/>
         <inertia ixx="2.94983710615554e-05" ixy="8.65358355557671e-09" ixz="-5.99019648532088e-09" iyy="3.11696241448887e-05" iyz="1.32416975855121e-06" izz="2.3568380981746e-05"/>
       </inertial>
@@ -30,5 +31,6 @@
       <inertial>
         <origin xyz="0.0315627099580794 3.23428430836527e-05 0.000305100560390667" rpy="0.0 -0.0 0.0"/>
-        <mass value="0.0155927868590324"/>
+        <!-- <mass value="0.0155927868590324"/> -->
+	<mass value="0.0215643963885794"/>
         <inertia ixx="4.31040540970899e-06" ixy="-1.84501397306783e-10" ixz="1.71628424283485e-09" iyy="2.33860081225919e-06" iyz="5.31064452921531e-10" izz="2.37493267246664e-06"/>
       </inertial>

File: robots/gimbalrotor/urdf/grape_with_arm/xacro/vial_pick_module.xacro (robot description, xacro)
@@ -10,6 +10,14 @@
       <inertial>
         <origin xyz="-8.31656604743406e-05 6.17407712109358e-07 0.0172789824004518" rpy="0.0 -0.0 0.0"/>
-        <mass value="0.0367410396327177"/>
-        <inertia ixx="2.74000444301134e-05" ixy="2.05651795964491e-09" ixz="1.05170944657198e-08" iyy="3.92773312962098e-06" iyz="1.41490289935768e-10" izz="2.96000106477188e-05"/>
+        <!-- <mass value="0.0367410396327177"/> -->
+	<mass value="0.0729671799"/>
+        <!-- <inertia ixx="2.74000444301134e-05" ixy="2.05651795964491e-09" ixz="1.05170944657198e-08" iyy="3.92773312962098e-06" iyz="1.41490289935768e-10" izz="2.96000106477188e-05"/> -->
+	<inertia
+	    ixx="5.44160968549e-05"
+	    ixy="4.08421529247e-09"
+	    ixz="2.08867993823e-08"
+	    iyy="7.80042189154e-06"
+	    iyz="2.80997694760e-10"
+	    izz="5.87851983387e-05"/>
       </inertial>
       <visual>
@@ -30,5 +38,6 @@
       <inertial>
         <origin xyz="-0.000120038522656072 -5.20570211972105e-12 -0.0147957403917136" rpy="0.0 -0.0 0.0"/>
-        <mass value="0.00343282009982582"/>
+        <!-- <mass value="0.00343282009982582"/> -->
+	<mass value="0.085"/>
         <inertia ixx="1.16286941033441e-07" ixy="8.67661870278422e-18" ixz="-1.77466824391762e-09" iyy="1.07255119256354e-07" iyz="-3.37024679420742e-17" izz="1.22297072354454e-07"/>
       </inertial>
@@ -51,5 +60,12 @@
         <origin xyz="-0.00786415967836717 -0.0219871091816924 0.0229800428255594" rpy="0.0 -0.0 0.0"/>
         <mass value="0.0266986294658226"/>
-        <inertia ixx="3.98880329468621e-06" ixy="1.86640977240353e-07" ixz="-1.1651136084322e-07" iyy="4.301768396309e-06" iyz="2.46993792736072e-07" izz="3.1771479602296e-06"/>
+        <!-- <inertia ixx="3.98880329468621e-06" ixy="1.86640977240353e-07" ixz="-1.1651136084322e-07" iyy="4.301768396309e-06" iyz="2.46993792736072e-07" izz="3.1771479602296e-06"/> -->
+	<inertia
+	    ixx="1.26990893103e-05"
+	    ixy="5.94205896813e-07"
+	    ixz="-3.70935357725e-07"
+	    iyy="1.36954713033e-05"
+	    iyz="7.86350191100e-07"
+	    izz="1.01150351918e-05"/>
       </inertial>
       <visual>
@@ -70,6 +86,14 @@
       <inertial>
         <origin xyz="0.00786416008938544 0.0219871091816897 0.0236476776647334" rpy="0.0 -0.0 0.0"/>
-        <mass value="0.0266986294658226"/>
-        <inertia ixx="3.9888032946862e-06" ixy="1.86636813590827e-07" ixz="1.16511360843049e-07" iyy="4.301768396309e-06" iyz="-9.59549183617184e-08" izz="3.1771479602296e-06"/>
+        <!-- <mass value="0.0266986294658226"/> -->
+	<mass value="0.085"/>
+        <!-- <inertia ixx="3.9888032946862e-06" ixy="1.86636813590827e-07" ixz="1.16511360843049e-07" iyy="4.301768396309e-06" iyz="-9.59549183617184e-08" izz="3.1771479602296e-06"/> -->
+	<inertia
+	    ixx="1.26990893103e-05"
+	    ixy="5.94192641069e-07"
+	    ixz="3.70935357725e-07"
+	    iyy="1.36954713033e-05"
+	    iyz="-3.05490140278e-07"
+	    izz="1.01150351918e-05"/>
       </inertial>
       <visual>

Commit message: [grape_with_arm] update gimbalrotor masparamators

File: robots/gimbalrotor/urdf/grape_with_arm/gimbalrotor.urdf.xacro (robot description, xacro)
@@ -53,7 +53,9 @@
   <link name="main_body">
     <inertial>
-      <origin xyz="-0.0041019 0.0000721 -0.0183334" rpy="0.0 -0.0 0.0"/>
+      <!-- <origin xyz="-0.0041019 0.0000721 -0.0183334" rpy="0.0 -0.0 0.0"/> -->
+      <origin xyz="0.0178508 0.0018366 -0.03525" rpy="0.0 -0.0 0.0"/>
       <!-- <mass value="1.3193189"/> -->
-      <mass value="2.0421872"/>
+      <!-- <mass value="2.0421872">/ -->
+      <mass value="1.8654999"/>
       <!-- <inertia ixx="0.0150906" ixy="-0.0000095" ixz="-0.0001112" iyy="0.0153469" iyz="-0.0000102" izz="0.0122100"/> -->
       <inertia
@@ -75,5 +77,6 @@
       <geometry>
         <!-- <mesh filename="package://gimbalrotor/urdf/grape/meshes/main_body.stl"/> -->
-        <box size="0.25 0.25 0.035"/>
+        <!-- <box size="0.25 0.25 0.035"/> -->
+	<box size="0.5 0.5 0.035"/>
       </geometry>
       <origin xyz="0.0 0.0 0.0" rpy="0.0 -0.0 0.0"/>
@@ -83,5 +86,6 @@
     <inertial>
       <origin xyz="0.0097185 -0.0000023 0.0115030" rpy="0.0 -0.0 0.0"/>
-      <mass value="0.2647482"/>
+      <!-- <mass value="0.2647482"/> -->
+      <mass value="0.308825311849623"/>
       <inertia ixx="0.0004342" ixy="0.0000000" ixz="-0.0000960" iyy="0.0005399" iyz="0.0000000" izz="0.0001644"/>
     </inertial>
@@ -112,5 +116,6 @@
     <inertial>
       <origin xyz="0.0097185 -0.0000023 0.0115030" rpy="0.0 -0.0 0.0"/>
-      <mass value="0.2647482"/>
+      <!-- <mass value="0.2647482"/> -->
+      <mass value="0.308825311849623"/>
       <inertia ixx="0.0004342" ixy="0.0000000" ixz="-0.0000960" iyy="0.0005399" iyz="0.0000000" izz="0.0001644"/>
     </inertial>
@@ -141,5 +146,6 @@
     <inertial>
       <origin xyz="0.0097185 -0.0000023 0.0115030" rpy="0.0 -0.0 0.0"/>
-      <mass value="0.2647482"/>
+      <!-- <mass value="0.2647482"/> -->
+      <mass value="0.308825311849623"/>
       <inertia ixx="0.0004342" ixy="0.0000000" ixz="-0.0000960" iyy="0.0005399" iyz="0.0000000" izz="0.0001644"/>
     </inertial>
@@ -170,5 +176,6 @@
     <inertial>
       <origin xyz="0.0097185 -0.0000023 0.0115030" rpy="0.0 -0.0 0.0"/>
-      <mass value="0.2647482"/>
+      <!-- <mass value="0.2647482"/> -->
+      <mass value="0.308825311849623"/>
       <inertia ixx="0.0004342" ixy="0.0000000" ixz="-0.0000960" iyy="0.0005399" iyz="0.0000000" izz="0.0001644"/>
     </inertial>

Commit message: [grape_with_arm] tmp update for test gimbalrotor

File: robots/gimbalrotor/urdf/grape_with_arm/gimbalrotor.urdf.xacro (robot description, xacro)
@@ -2,5 +2,5 @@
 <robot name="gimbalrotor" xmlns:xacro="http://www.ros.org/wiki/xacro">
   <xacro:include filename="$(find gimbalrotor)/urdf/grape_with_arm/common.xacro"/>
-  <xacro:include filename="$(find gimbalrotor)/urdf/grape_with_arm/xacro/arm.xacro"/>
+  <!-- <xacro:include filename="$(find gimbalrotor)/urdf/grape_with_arm/xacro/arm.xacro"/> -->
   <!-- <link name="root"> -->
   <!--   <inertial> -->
@@ -240,5 +240,5 @@
   <!-- </joint> -->
   <joint name="gimbal1" type="revolute">
-    <limit effort="5.0" velocity="10.0" lower="-3.14" upper="3.14"/>
+    <limit effort="1.5" velocity="6.39" lower="-3.14" upper="3.14"/>
     <parent link="main_body"/>
     <child link="gimbal1_link"/>
@@ -254,5 +254,5 @@
   </joint>
   <joint name="gimbal2" type="revolute">
-    <limit effort="5.0" velocity="10.0" lower="-3.14" upper="3.14"/>
+    <limit effort="1.5" velocity="6.39" lower="-3.14" upper="3.14"/>
     <parent link="main_body"/>
     <child link="gimbal2_link"/>
@@ -268,5 +268,5 @@
   </joint>
   <joint name="gimbal3" type="revolute">
-    <limit effort="5.0" velocity="10.0" lower="-3.14" upper="3.14"/>
+    <limit effort="1.5" velocity="6.39" lower="-3.14" upper="3.14"/>
     <parent link="main_body"/>
     <child link="gimbal3_link"/>
@@ -282,5 +282,5 @@
   </joint>
   <joint name="gimbal4" type="revolute">
-    <limit effort="5.0" velocity="10.0" lower="-3.14" upper="3.14"/>
+    <limit effort="1.5" velocity="6.39" lower="-3.14" upper="3.14"/>
     <parent link="main_body"/>
     <child link="gimbal4_link"/>
@@ -405,4 +405,5 @@
   <!--   <inertial> -->
   <!--     <origin xyz="0 0 0" rpy="0 0 0"/> -->
+  <!--     <mass value="0.0001"/> -->
   <!--     <mass value="1.1"/> -->
   <!--     <inertia -->
@@ -417,5 +418,5 @@
   <!--   <origin xyz="0 0 -0.08" rpy="3.14159 0 0"/> -->
   <!-- </joint> -->
-  <!-- Include the arm macro -->
-  <xacro:arm parent_link="main_body"/>
+  <!-- <!-\- Include the arm macro -\-> -->
+  <!-- <xacro:arm parent_link="main_body"/> -->
 </robot>

File: robots/gimbalrotor/urdf/grape_with_arm/xacro/arm.xacro (robot description, xacro)
@@ -7,5 +7,5 @@
   <xacro:include filename="$(find gimbalrotor)/urdf/grape_with_arm/xacro/screw_drive_module_dynamixel.xacro"/>
   <xacro:include filename="$(find gimbalrotor)/urdf/grape_with_arm/xacro/vial_pick_module.xacro"/>
-  <xacro:macro name="arm" params="parent_link:=main_body xyz:='0.0995 0.0 -0.046' rpy:='3.141592653589793 1.5707926535897934 3.141592653589793'">
+  <xacro:macro name="arm" params="parent_link:=main_body xyz:='0.0995 0.0 -0.0465' rpy:='3.141592653589793 1.5707926535897934 3.141592653589793'">
     <!-- Dummy link to attach the arm to the main body -->
     <link name="arm_dummy_link"/>
