Commit message: change fanguard param

File: robots/gimbalrotor/urdf/grape_with_arm/gimbalrotor.urdf.xacro (robot description, xacro)
@@ -2,4 +2,5 @@
 <robot name="gimbalrotor" xmlns:xacro="http://www.ros.org/wiki/xacro">
   <xacro:include filename="$(find gimbalrotor)/urdf/grape_with_arm/common.xacro"/>
+  <xacro:include filename="$(find gimbalrotor)/urdf/grape_with_arm/xacro/gimbal_inertial.xacro"/>
   <xacro:include filename="$(find gimbalrotor)/urdf/grape_with_arm/xacro/arm.xacro"/>
   <!-- <link name="root"> -->
@@ -84,10 +85,5 @@
   </link>
   <link name="gimbal1_link">
-    <inertial>
-      <origin xyz="0.0097185 -0.0000023 0.0115030" rpy="0.0 -0.0 0.0"/>
-      <!-- <mass value="0.2647482"/> -->
-      <mass value="0.308825311849623"/>
-      <inertia ixx="0.0004342" ixy="0.0000000" ixz="-0.0000960" iyy="0.0005399" iyz="0.0000000" izz="0.0001644"/>
-    </inertial>
+    <xacro:gimbal_module_inertial/>
     <visual>
       <geometry>
@@ -114,10 +110,5 @@
   </link>
   <link name="gimbal2_link">
-    <inertial>
-      <origin xyz="0.0097185 -0.0000023 0.0115030" rpy="0.0 -0.0 0.0"/>
-      <!-- <mass value="0.2647482"/> -->
-      <mass value="0.308825311849623"/>
-      <inertia ixx="0.0004342" ixy="0.0000000" ixz="-0.0000960" iyy="0.0005399" iyz="0.0000000" izz="0.0001644"/>
-    </inertial>
+    <xacro:gimbal_module_inertial/>
     <visual>
       <geometry>
@@ -144,10 +135,5 @@
   </link>
   <link name="gimbal3_link">
-    <inertial>
-      <origin xyz="0.0097185 -0.0000023 0.0115030" rpy="0.0 -0.0 0.0"/>
-      <!-- <mass value="0.2647482"/> -->
-      <mass value="0.308825311849623"/>
-      <inertia ixx="0.0004342" ixy="0.0000000" ixz="-0.0000960" iyy="0.0005399" iyz="0.0000000" izz="0.0001644"/>
-    </inertial>
+    <xacro:gimbal_module_inertial/>
     <visual>
       <geometry>
@@ -174,10 +160,5 @@
   </link>
   <link name="gimbal4_link">
-    <inertial>
-      <origin xyz="0.0097185 -0.0000023 0.0115030" rpy="0.0 -0.0 0.0"/>
-      <!-- <mass value="0.2647482"/> -->
-      <mass value="0.308825311849623"/>
-      <inertia ixx="0.0004342" ixy="0.0000000" ixz="-0.0000960" iyy="0.0005399" iyz="0.0000000" izz="0.0001644"/>
-    </inertial>
+    <xacro:gimbal_module_inertial/>
     <visual>
       <geometry>

Commit message: update

File: robots/gimbalrotor/urdf/grape_with_arm/gimbalrotor.urdf.xacro (robot description, xacro)
@@ -59,5 +59,6 @@
       <!-- <mass value="1.3193189"/> -->
       <!-- <mass value="2.0421872">/ -->
-      <mass value="1.8654999"/>
+      <!-- <mass value="1.8654999"/> -->
+      <mass value="2.489"/>
       <!-- <inertia ixx="0.0150906" ixy="-0.0000095" ixz="-0.0001112" iyy="0.0153469" iyz="-0.0000102" izz="0.0122100"/> -->
       <inertia
